File: 39D/39D.kicad_pcb (KiCad board)
At the start: 2 copper layers, 10.7 x 10.7 mm, 11 parts, among them J1 Conn_01x04, J2 Conn_01x04

Commit message: apdate all footprints an run drc
Parts:
- G***: footprint LOGO -> Library:LOGO
- moved D2 0.09 mm to (120.0, 97.3)
